Commit message: feat(urdf)增加正方体可视化

File: src/my_tf_tree/urdf/r2.urdf.xacro (robot description, xacro)
@@ -3,5 +3,15 @@
   <xacro:property name="PI" value="3.1415926535897931" />
   <!-- base_link -->
-  <link name="base_link" />
+  <link name="base_link">
+    <visual>
+      <geometry>
+        <box size="0.5 0.5 0.2"/>
+      </geometry>
+      <origin xyz="0 0 0.1" rpy="0 0 0"/>
+      <material name="purple">
+        <color rgba="0.5 0 0.5 1"/> <!-- 紫色 -->
+      </material>
+    </visual>
+  </link>
   <!-- laser_frame attached to base_link -->
   <link name="laser_frame" />

Commit message: 更改tf与imu 适配

File: src/my_tf_tree/urdf/r2.urdf.xacro (robot description, xacro)
@@ -19,5 +19,5 @@
     <parent link="base_link" />
     <child link="laser_frame" />
-    <origin xyz="-0.1 0 0" rpy="0 0 0" />
+    <origin xyz="0.2 0 0" rpy="0 0 0" />
   </joint>
   <!-- livox_frame attached to base_link -->
@@ -26,5 +26,5 @@
     <parent link="base_link" />
     <child link="livox_frame" />
-    <origin xyz="0 0 0" rpy="0 0 0" />
+    <origin xyz="0.15 -0.2 0" rpy="0 0 0" />
   </joint>
 </robot>
